File: pcb/ai_hat_proto.brd (EAGLE design)
At the start: 65 x 56 mm, 285 parts, among them J1 1X01-SM, J10 1X01-SM, J100 1X01-SM, J101 1X01-SM, J102 1X01-SM, J103 1X01-SM, J104 1X01-SM, J105 1X01-SM, J106 1X01-SM, J107 1X01-SM, J108 1X01-SM, J109 1X01-SM, J11 1X01-SM, J110 1X01-SM, J111 1X01-SM, J112 1X01-SM, J113 1X01-SM, J114 1X01-SM, J115 1X01-SM, J116 1X01-SM, J117 1X01-SM, J118 1X01-SM, J119 1X01-SM, J12 1X01-SM, J120 1X01-SM, J121 1X01-SM, J122 1X01-SM, J123 1X01-SM, J124 1X01-SM, J125 1X01-SM, J126 1X01-SM, J127 1X01-SM, J128 1X01-SM, J129 1X01-SM, J13 1X01-SM, J130 1X01-SM, J131 1X01-SM, J132 1X01-SM, J133 1X01-SM, J134 1X01-SM, J135 1X01-SM, J136 1X01-SM, J137 1X01-SM, J138 1X01-SM, J139 1X01-SM, J14 1X01-SM, J140 1X01-SM, J141 1X01-SM, J142 1X01-SM, J143 1X01-SM, J144 1X01-SM, J145 1X01-SM, J146 1X01-SM, J147 1X01-SM, J148 1X01-SM, J149 1X01-SM, J15 1X01-SM, J150 1X01-SM, J151 1X01-SM, J152 1X01-SM, J153 1X01-SM, J154 1X01-SM, J155 1X01-SM, J156 1X01-SM, J157 1X01-SM, J158 1X01-SM, J159 1X01-SM, J16 1X01-SM, J160 1X01-SM, J161 1X01-SM, J162 1X01-SM, J163 1X01-SM, J164 1X01-SM, J165 1X01-SM, J166 1X01-SM, J167 1X01-SM, J168 1X01-SM, J169 1X01-SM, J17 1X01-SM, J170 1X01-SM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

Commit message: updating
Parts:
- moved U$9 0.51 mm to (3.17, 17.1)
Routing:
- net MOSI: track 50.7 -> 51.4 mm
Other:
- board text added: "PROTO HAT for Raspberry Pi A+/B+/2"
- board text removed: "PROTO HAT for Raspberry Pi A+/B+"
Changed lines of the file:
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@@
 <layer number="56" name="wert" color="7" fill="1" visible="no" active="no"/>
 <layer number="57" name="tCAD" color="7" fill="1" visible="no" active="no"/>
+<layer number="90" name="Modules" color="5" fill="1" visible="no" active="no"/>
 <layer number="91" name="Nets" color="2" fill="1" visible="no" active="no"/>
 <layer number="92" name="Busses" color="1" fill="1" visible="no" active="no"/>
@@
 <layer number="251" name="SMDround" color="12" fill="11" visible="no" active="no"/>
 <layer number="254" name="cooling" color="7" fill="1" visible="yes" active="yes"/>
+<layer number="255" name="routoute" color="7" fill="1" visible="yes" active="yes"/>
 </layers>
 <board>
@@
 <text x="57.404" y="3.175" size="1.27" layer="21" font="vector" ratio="10" rot="R180">GND</text>
 <wire x1="6.858" y1="21.463" x2="53.086" y2="21.463" width="0.4064" layer="21"/>
-<text x="47.244" y="37.465" size="1.27" layer="21" font="vector" ratio="10" rot="R180">PROTO HAT for Raspberry Pi A+/B+</text>
+<text x="48.514" y="37.465" size="1.27" layer="21" font="vector" ratio="10" rot="R180">PROTO HAT for Raspberry Pi A+/B+/2</text>
 <text x="7.874" y="36.957" size="0.762" layer="21" font="vector" ratio="10" rot="R180">v1.0</text>
 <text x="4.826" y="6.604" size="0.9144" layer="21" font="vector" ratio="10" rot="R90">www.acrobotic.com</text>
@@
 <attribute name="NAME" x="56.769" y="7.112" size="1.016" layer="25" font="vector" ratio="10" rot="R90"/>
 </element>
-<element name="U$9" library="Ai_Miscellany" package="AI-LOGO-XS" value="AI-LOGOXS" x="3.175" y="16.637" rot="R90"/>
+<element name="U$9" library="Ai_Miscellany" package="AI-LOGO-XS" value="AI-LOGOXS" x="3.175" y="17.145" rot="R90"/>
 <element name="U$10" library="Ai_Miscellany" package="AI-LOGO-XS" value="AI-LOGOXS" x="3.175" y="19.177" rot="MR270"/>
 </elements>
@@
 <wire x1="58.022" y1="35.941" x2="61.722" y2="35.941" width="0.254" layer="1"/>
 <via x="61.722" y="35.941" extent="1-16" drill="0.508"/>
-<wire x1="61.722" y1="35.941" x2="31.496" y2="35.941" width="0.254" layer="16"/>
-<via x="31.496" y="35.941" extent="1-16" drill="0.508"/>
-<wire x1="31.496" y1="35.941" x2="31.115" y2="36.322" width="0.254" layer="1"/>
-<wire x1="31.115" y1="36.322" x2="31.115" y2="43.561" width="0.254" layer="1"/>
+<wire x1="61.722" y1="35.941" x2="61.341" y2="35.56" width="0.254" layer="16"/>
+<wire x1="61.341" y1="35.56" x2="31.242" y2="35.56" width="0.254" layer="16"/>
+<via x="31.242" y="35.56" extent="1-16" drill="0.508"/>
+<wire x1="31.242" y1="35.56" x2="31.115" y2="35.687" width="0.254" layer="1"/>
+<wire x1="31.115" y1="35.687" x2="31.115" y2="43.561" width="0.254" layer="1"/>
 <wire x1="31.115" y1="43.561" x2="30.226" y2="44.45" width="0.254" layer="1"/>
 <wire x1="30.226" y1="44.45" x2="29.845" y2="44.45" width="0.254" layer="1"/>

Commit message: changed resistor value
Parts:
- R4: value 300 -> 330
Changed lines of the file:
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@@
 <setting verticaltext="up"/>
 </settings>
-<grid distance="5" unitdist="mil" unit="mil" style="lines" multiple="1" display="yes" altdistance="0.025" altunitdist="inch" altunit="inch"/>
+<grid distance="50" unitdist="mil" unit="mil" style="lines" multiple="1" display="yes" altdistance="0.025" altunitdist="inch" altunit="inch"/>
 <layers>
 <layer number="1" name="Top" color="4" fill="1" visible="yes" active="yes"/>
@@
 <element name="CFG" library="Ai_Connectors" package="1X02-SJ-NO" value="1X02-SJ-NO" x="55.753" y="16.637" rot="R90"/>
 <element name="J19" library="Ai_Connectors" package="JST-4P-SMD" value="JST-4P-MALE" x="61.976" y="36.957" rot="R270"/>
-<element name="R4" library="Ai_Passives" package="RES-0603" value="300" x="54.864" y="7.62" smashed="yes" rot="R90">
+<element name="R4" library="Ai_Passives" package="RES-0603" value="330" x="54.864" y="7.62" smashed="yes" rot="R90">
 <attribute name="NAME" x="56.769" y="7.112" size="1.016" layer="25" font="vector" ratio="10" rot="R90"/>
 </element>

Commit message: updating
Parts:
- added FRAME1: FRAME-LETTER, Ai_Miscellany:CREATIVE-COMMONS
- C1: value 100nF -> 0.1uF
- R1, R2: value 3k9 -> 3K9
- R3: value 1k -> 1K
- moved U$10 1.89 mm to (1.91, 17.8)
- moved U$9 1.42 mm to (1.91, 17.8)
Other:
- board text added: "19"
- board text added: "@MakerBro"
- board text removed: "15"
